File: controller.sch (KiCad schematic (older format))
At the start: 29 parts, among them Q1 Q_PMOS_SGD, Q2 Q_PMOS_SGD, SW1 L1, SW2 L2, SW3 Select, SW4 Start, SW5 R2, SW6 R1, U5 ProMicro

Commit message: Create 5pos switch thumbstick FPC connector.
Based off TE 5pos 0.5mm pitch connector.
Parts:
- F1, F2: footprint (none) -> rpi-shell-v1-sockets:046809605110846+
Changed lines of the file:
@@
 F 0 "F1" H 2100 2350 50  0000 C CNN
 F 1 "046809605110846+" H 2133 3174 50  0000 C CNN
-F 2 "" H 2100 3000 50  0001 C CNN
+F 2 "rpi-shell-v1-sockets:046809605110846+" H 2100 3000 50  0001 C CNN
 F 3 "" H 2100 3000 50  0001 C CNN
 	1    2100 2850
@@
 F 0 "F2" H 9500 3400 50  0000 R CNN
 F 1 "046809605110846+" H 9840 2532 50  0000 R CNN
-F 2 "" H 9450 3200 50  0001 C CNN
+F 2 "rpi-shell-v1-sockets:046809605110846+" H 9450 3200 50  0001 C CNN
 F 3 "" H 9450 3200 50  0001 C CNN
 	1    9450 3050

Commit message: Update symbols to remove layout warnings.
Change shoulder button switches to SPST (two pin) switches to match the
side actuated devices. Change the speaker symbol pin names to '+' and
'-' to match the footprint.
Parts:
- SW1, SW2, SW5, SW6: symbol Switch:SW_MEC_5E -> Switch:SW_SPST
Connections:
- wire segments 97 -> 98
- no-connect marks 22 -> 14
Other:
- moved on the sheet: SW3
Changed lines of the file:
@@
 $EndComp
 $Comp
-L Switch:SW_MEC_5E SW1
-U 1 1 60680B20
-P 1850 1200
-F 0 "SW1" H 1850 1585 50  0000 C CNN
-F 1 "L1" H 1850 1494 50  0000 C CNN
-F 2 "rpi-shell-v1-switches:MJTP1236" H 1850 1500 50  0001 C CNN
-F 3 "http://www.apem.com/int/index.php?controller=attachment&id_attachment=1371" H 1850 1500 50  0001 C CNN
-	1    1850 1200
-	1    0    0    -1
-$EndComp
-$Comp
-L Switch:SW_MEC_5E SW3
-U 1 1 60680B26
-P 3500 1200
-F 0 "SW3" H 3500 1585 50  0000 C CNN
-F 1 "Select" H 3500 1494 50  0000 C CNN
-F 2 "rpi-shell-v1-switches:SW_SMD_Dome_TL3312NF-160Q" H 3500 1500 50  0001 C CNN
-F 3 "http://www.apem.com/int/index.php?controller=attachment&id_attachment=1371" H 3500 1500 50  0001 C CNN
-	1    3500 1200
-	1    0    0    -1
-$EndComp
-$Comp
-L Switch:SW_MEC_5E SW2
+L Switch:SW_SPST SW2
 U 1 1 60680B2C
-P 2700 1200
-F 0 "SW2" H 2700 1585 50  0000 C CNN
-F 1 "L2" H 2700 1494 50  0000 C CNN
-F 2 "rpi-shell-v1-switches:MJTP1236" H 2700 1500 50  0001 C CNN
-F 3 "http://www.apem.com/int/index.php?controller=attachment&id_attachment=1371" H 2700 1500 50  0001 C CNN
-	1    2700 1200
-	1    0    0    -1
-$EndComp
-$Comp
-L Switch:SW_MEC_5E SW5
+P 2700 1250
+F 0 "SW2" H 2700 1500 50  0000 C CNN
+F 1 "L2" H 2700 1400 50  0000 C CNN
+F 2 "rpi-shell-v1-switches:MJTP1236" H 2700 1550 50  0001 C CNN
+F 3 "http://www.apem.com/int/index.php?controller=attachment&id_attachment=1371" H 2700 1550 50  0001 C CNN
+	1    2700 1250
+	1    0    0    -1
+$EndComp
+$Comp
+L Switch:SW_SPST SW5
 U 1 1 60680B32
 P 8900 1300
-F 0 "SW5" H 8900 1685 50  0000 C CNN
-F 1 "R2" H 8900 1594 50  0000 C CNN
+F 0 "SW5" H 8900 1550 50  0000 C CNN
+F 1 "R2" H 8900 1450 50  0000 C CNN
 F 2 "rpi-shell-v1-switches:MJTP1236" H 8900 1600 50  0001 C CNN
 F 3 "http://www.apem.com/int/index.php?controller=attachment&id_attachment=1371" H 8900 1600 50  0001 C CNN
@@
 $EndComp
 Wire Wire Line
-	1650 1200 1500 1200
-Wire Wire Line
-	1500 1200 1500 1350
-Wire Wire Line
-	2500 1200 2500 1350
-Wire Wire Line
-	2500 1350 1500 1350
-Wire Wire Line
-	3300 1200 3300 1350
+	1650 1250 1600 1250
+Wire Wire Line
+	1600 1250 1600 1350
+Wire Wire Line
+	2500 1250 2500 1350
+Wire Wire Line
+	2500 1350 1600 1350
+Wire Wire Line
+	3300 1250 3300 1350
 Wire Wire Line
 	3300 1350 2500 1350
@@
 $EndComp
 Wire Wire Line
-	3700 1200 3700 1500
-Wire Wire Line
-	2900 1200 2900 1500
-Wire Wire Line
-	2050 1200 2050 1500
+	3700 1250 3700 1500
+Wire Wire Line
+	2900 1250 2900 1500
+Wire Wire Line
+	2050 1250 2050 1500
 Wire Wire Line
 	3300 1350 4300 1350
@@
 Connection ~ 9100 1400
 Wire Wire Line
-	9100 1400 9850 1400
+	9100 1400 9900 1400
 Wire Wire Line
 	8350 1300 8350 1400
@@
 Wire Wire Line
 	8400 3050 8050 3050
-NoConn ~ 1650 1100
-NoConn ~ 2050 1100
-NoConn ~ 2500 1100
-NoConn ~ 2900 1100
-NoConn ~ 3300 1100
-NoConn ~ 3700 1100
-Wire Wire Line
-	9850 1400 9850 1300
+Wire Wire Line
+	9900 1400 9900 1300
 Wire Wire Line
 	9450 1300 9450 1500
 $Comp
-L Switch:SW_MEC_5E SW6
+L Switch:SW_SPST SW6
 U 1 1 60680BB6
 P 9650 1300
-F 0 "SW6" H 9650 1685 50  0000 C CNN
-F 1 "R1" H 9650 1594 50  0000 C CNN
+F 0 "SW6" H 9650 1550 50  0000 C CNN
+F 1 "R1" H 9650 1450 50  0000 C CNN
 F 2 "rpi-shell-v1-switches:MJTP1236" H 9650 1600 50  0001 C CNN
 F 3 "http://www.apem.com/int/index.php?controller=attachment&id_attachment=1371" H 9650 1600 50  0001 C CNN
@@
 	1    0    0    -1
 $EndComp
-NoConn ~ 9850 1200
-NoConn ~ 9450 1200
-NoConn ~ 9100 1200
-NoConn ~ 8700 1200
 NoConn ~ 8350 1200
 NoConn ~ 7950 1200
+$Comp
+L Switch:SW_SPST SW1
+U 1 1 60680B20
+P 1850 1250
+F 0 "SW1" H 1850 1500 50  0000 C CNN
+F 1 "L1" H 1850 1400 50  0000 C CNN
+F 2 "rpi-shell-v1-switches:MJTP1236" H 1850 1550 50  0001 C CNN
+F 3 "http://www.apem.com/int/index.php?controller=attachment&id_attachment=1371" H 1850 1550 50  0001 C CNN
+	1    1850 1250
+	1    0    0    -1
+$EndComp
+NoConn ~ 3700 1150
+NoConn ~ 3300 1150
+$Comp
+L Switch:SW_MEC_5E SW3
+U 1 1 60680B26
+P 3500 1250
+F 0 "SW3" H 3500 1635 50  0000 C CNN
+F 1 "Select" H 3500 1544 50  0000 C CNN
+F 2 "rpi-shell-v1-switches:SW_SMD_Dome_TL3312NF-160Q" H 3500 1550 50  0001 C CNN
+F 3 "http://www.apem.com/int/index.php?controller=attachment&id_attachment=1371" H 3500 1550 50  0001 C CNN
+	1    3500 1250
+	1    0    0    -1
+$EndComp
+Wire Wire Line
+	9900 1300 9850 1300
 Wire Bus Line
 	5850 2100 9900 2100

Commit message: Add 3ds button cross footprint.
Parts:
- CT1: footprint (none) -> rpi-shell-v1-switches:3ds_dpad_cross
Changed lines of the file:
@@
 F 0 "CT1" H 2750 6215 50  0000 C CNN
 F 1 "dpad-cross-trace" H 2750 6124 50  0000 C CNN
-F 2 "" H 2800 4400 50  0001 C CNN
+F 2 "rpi-shell-v1-switches:3ds_dpad_cross" H 2800 4400 50  0001 C CNN
 F 3 "" H 2800 4400 50  0001 C CNN
 	1    2800 5450
